File: hardware/kicad/pi-cemaker.kicad_sch (KiCad schematic)
At the start: 0 parts

Commit message: hardware: draft Lite board generated from design.py (ERC clean, PCB unrouted/unreviewed)
Schematic (110 parts, ERC 0 violations), hand-built BQ25792 footprint,
placed + autorouted draft PCB (38 connections unrouted), draft BOM and a
decision log with a reversal path for each guess. No fab files produced.

Co-Authored-By: Claude Sonnet 5.5 <noreply@anthropic.com>
Parts:
- added C1: 1uF 25V, Capacitor_SMD:C_0603_1608Metric, symbol Device:C
- added C10, C9: 47nF 25V, Capacitor_SMD:C_0603_1608Metric, symbol Device:C
- added C11: 4.7uF 10V, Capacitor_SMD:C_0805_2012Metric, symbol Device:C
- added C12, C13, C14, C15, C16, C2, C22, C23, C3, C5, C6, C7: 10uF 25V, Capacitor_SMD:C_1206_3216Metric, symbol Device:C
- added C17, C24, C4, C8: 100nF 25V, Capacitor_SMD:C_0603_1608Metric, symbol Device:C
- added C18, C19: 10uF 16V, Capacitor_SMD:C_1206_3216Metric, symbol Device:C
- added C20: 1nF 50V, Capacitor_SMD:C_0603_1608Metric, symbol Device:C
- added C21: 100nF 16V, Capacitor_SMD:C_0603_1608Metric, symbol Device:C
- added C25, C26: 33uF 16V, Capacitor_SMD:C_1210_3225Metric, symbol Device:C
- added C27, C28: 33uF 16V (spare), Capacitor_SMD:C_1210_3225Metric, symbol Device:C
- added C29: 33pF (CFF), Capacitor_SMD:C_0603_1608Metric, symbol Device:C
- added C30: 10uF 10V, Capacitor_SMD:C_0805_2012Metric, symbol Device:C
- added D1: SMAJ13A, Diode_SMD:D_SMA, symbol Device:D_TVS
- added D2: SS34, Diode_SMD:D_SMA, symbol Device:D_Schottky
- added D3: green, LED_SMD:LED_0603_1608Metric, symbol Device:LED
- added D4: amber, LED_SMD:LED_0603_1608Metric, symbol Device:LED
- added D5: red, LED_SMD:LED_0603_1608Metric, symbol Device:LED
- added F1: 3.15A or 0R (fit one), Fuse:Fuse_1206_3216Metric, symbol Device:Fuse
- added H1, H2, H3, H4: M2.5, MountingHole:MountingHole_2.7mm_M2.5_Pad, symbol Mechanical:MountingHole
- added J1: USB-C in (PD sink), Connector_USB:USB_C_Receptacle_GCT_USB4105-xx-A_16P_TopMnt_Horizontal, symbol Connector:USB_C_Receptacle_USB2.0_16P
- added J2: USB-C out to Pi 5 (power only), Connector_USB:USB_C_Receptacle_GCT_USB4105-xx-A_16P_TopMnt_Horizontal, symbol Connector:USB_C_Receptacle_USB2.0_16P
- added J3: PACK+ / PACK- (off-board 2S BMS), TerminalBlock_Phoenix:TerminalBlock_Phoenix_MKDS-1,5-2_1x02_P5.00mm_Horizontal, symbol Connector_Generic:Conn_01x02
- added J4: 5V OUT / GND, TerminalBlock_Phoenix:TerminalBlock_Phoenix_MKDS-1,5-2_1x02_P5.00mm_Horizontal, symbol Connector_Generic:Conn_01x02
- added J5: To Pi 5 J2 power button, Connector_PinHeader_2.54mm:PinHeader_1x02_P2.54mm_Vertical, symbol Connector_Generic:Conn_01x02
- added J6: NTC (optional), Connector_PinHeader_2.54mm:PinHeader_1x02_P2.54mm_Vertical, symbol Connector_Generic:Conn_01x02
- added J7: I2C expansion (3V3 SDA), Connector_PinHeader_2.54mm:PinHeader_1x02_P2.54mm_Vertical, symbol Connector_Generic:Conn_01x02
- added JP1: VSYS link, Jumper:SolderJumper-2_P1.3mm_Bridged_RoundedPad1.0x1.5mm, symbol Jumper:SolderJumper_2_Bridged
- added JP2: 5V link, Jumper:SolderJumper-2_P1.3mm_Bridged_RoundedPad1.0x1.5mm, symbol Jumper:SolderJumper_2_Bridged
- added JP3: PACK link, Jumper:SolderJumper-2_P1.3mm_Bridged_RoundedPad1.0x1.5mm, symbol Jumper:SolderJumper_2_Bridged
- added L1: 1uH >=8A sat, Inductor_SMD:L_Bourns_SRP7028A_7.3x6.6mm, symbol Device:L
- added L2: 4.7uH >=8A sat, Inductor_SMD:L_Bourns_SRP7028A_7.3x6.6mm, symbol Device:L
- added Q1, Q2: 2N7002, Package_TO_SOT_SMD:SOT-23, symbol Transistor_FET:2N7002
- added R1: 10k (12 V), Resistor_SMD:R_0603_1608Metric, symbol Device:R
- added R10, R15, R19, R20, R9: 10k, Resistor_SMD:R_0603_1608Metric, symbol Device:R
- added R11: 102k (FBT), Resistor_SMD:R_0603_1608Metric, symbol Device:R
- added R12: 19.1k (FBB), Resistor_SMD:R_0603_1608Metric, symbol Device:R
- added R13: 62k (ENT), Resistor_SMD:R_0603_1608Metric, symbol Device:R
- added R14: 21.5k (ENB), Resistor_SMD:R_0603_1608Metric, symbol Device:R
- added R16, R24: 100k (gate pull-down), Resistor_SMD:R_0603_1608Metric, symbol Device:R
- added R17, R18: 10k (Rp, 3 A), Resistor_SMD:R_0603_1608Metric, symbol Device:R
- added R2: 22.6k (3 A), Resistor_SMD:R_0603_1608Metric, symbol Device:R
- added R21, R22, R23: 1k, Resistor_SMD:R_0603_1608Metric, symbol Device:R
- added R3: 6.04k 1% (2S,1.5MHz), Resistor_SMD:R_0603_1608Metric, symbol Device:R
- added R4: 10k (CE low = charge on), Resistor_SMD:R_0603_1608Metric, symbol Device:R
- added R5: 100R, Resistor_SMD:R_0603_1608Metric, symbol Device:R
- added R6: 5.24k (RT1), Resistor_SMD:R_0603_1608Metric, symbol Device:R
- added R7: 30.31k (RT2), Resistor_SMD:R_0603_1608Metric, symbol Device:R
- added R8: 10k fixed NTC stand-in, Resistor_SMD:R_0603_1608Metric, symbol Device:R
- added SW1: USER, Button_Switch_SMD:SW_SPST_PTS810, symbol Switch:SW_Push
- added TP1: VBUS, TestPoint:TestPoint_Pad_D1.0mm, symbol Connector:TestPoint
- added TP10: STAT, TestPoint:TestPoint_Pad_D1.0mm, symbol Connector:TestPoint
- added TP11: INT, TestPoint:TestPoint_Pad_D1.0mm, symbol Connector:TestPoint
- added TP12: PACK_P, TestPoint:TestPoint_Pad_D1.0mm, symbol Connector:TestPoint
- added TP13: SW_B, TestPoint:TestPoint_Pad_D1.0mm, symbol Connector:TestPoint
- added TP14: EN_B, TestPoint:TestPoint_Pad_D1.0mm, symbol Connector:TestPoint
- added TP15: V5_B, TestPoint:TestPoint_Pad_D1.0mm, symbol Connector:TestPoint
- added TP16: FB, TestPoint:TestPoint_Pad_D1.0mm, symbol Connector:TestPoint
- added TP17: PG, TestPoint:TestPoint_Pad_D1.0mm, symbol Connector:TestPoint
- added TP18: VSYS_B, TestPoint:TestPoint_Pad_D1.0mm, symbol Connector:TestPoint
- added TP19: V5, TestPoint:TestPoint_Pad_D1.0mm, symbol Connector:TestPoint
- added TP2: PMID, TestPoint:TestPoint_Pad_D1.0mm, symbol Connector:TestPoint
- added TP20: +3V3, TestPoint:TestPoint_Pad_D1.0mm, symbol Connector:TestPoint
- added TP21: SDA, TestPoint:TestPoint_Pad_D1.0mm, symbol Connector:TestPoint
- added TP22: SCL, TestPoint:TestPoint_Pad_D1.0mm, symbol Connector:TestPoint
- added TP23: RUN, TestPoint:TestPoint_Pad_D1.0mm, symbol Connector:TestPoint
- added TP24, TP25, TP26, TP27: GND, TestPoint:TestPoint_Pad_D1.0mm, symbol Connector:TestPoint
- added TP3: SW1, TestPoint:TestPoint_Pad_D1.0mm, symbol Connector:TestPoint
- added TP4: SW2, TestPoint:TestPoint_Pad_D1.0mm, symbol Connector:TestPoint
- added TP5: REGN, TestPoint:TestPoint_Pad_D1.0mm, symbol Connector:TestPoint
- added TP6: TS, TestPoint:TestPoint_Pad_D1.0mm, symbol Connector:TestPoint
- added TP7: QON, TestPoint:TestPoint_Pad_D1.0mm, symbol Connector:TestPoint
- added TP8: VSYS, TestPoint:TestPoint_Pad_D1.0mm, symbol Connector:TestPoint
- added TP9: BAT, TestPoint:TestPoint_Pad_D1.0mm, symbol Connector:TestPoint
- added U1: HUSB238, Package_DFN_QFN:DFN-10-1EP_3x3mm_P0.5mm_EP1.65x2.38mm, symbol Interface_USB:HUSB238_xxxDD
- added U2: BQ25792, pi-cemaker:VQFN-HR-29_RQM0029A_4x4mm, symbol pi-cemaker:BQ25792
- added U3: LMR51450SDRRR, Package_SON:WSON-12-1EP_3x3mm_P0.5mm_EP1.5x2.5mm, symbol pi-cemaker:LMR51450
- added U4: Raspberry Pi Pico (RP2040), Module:RaspberryPi_Pico_Common_THT, symbol MCU_Module:RaspberryPi_Pico
Connections:
- net USB_DM: now also J1.A7 (D-), J1.B7 (D-), U1.3 (D-)
- net USB_DP: now also J1.A6 (D+), J1.B6 (D+), U1.2 (D+)
- new net +3V3: R10.2, R15.2, R19.2, R20.2, R9.2, TP20.1, U4.36 (3V3)
- new net BAT: C18.1, C19.1, JP3.2 (B), TP9.1, U2.22 (BAT), U2.23 (BAT)
- new net BATP: R5.2, U2.18 (BATP)
- new net BOOT_B: C21.1, U3.4 (BOOT)
- new net BTST1: C9.1, U2.4 (BTST1)
- new net BTST2: C10.1, U2.19 (BTST2)
- new net CC1_IN: J1.A5 (CC1), U1.4 (CC1)
- new net CC1_OUT: J2.A5 (CC1), R17.2
- new net CC2_IN: J1.B5 (CC2), U1.5 (CC2)
- new net CC2_OUT: J2.B5 (CC2), R18.2
- new net CE: R4.1, U2.13 (CE)
- new net EN_B: Q1.3 (D), R13.2, R14.1, TP14.1, U3.9 (EN)
- new net EN_KILL: Q1.1 (G), R16.1, U4.20 (GPIO15)
- new net FB: C29.2, R11.2, R12.1, TP16.1, U3.7 (FB)
- new net GND: C1.2, C11.2, C12.2, C13.2, C14.2, C15.2, C16.2, C17.2, C18.2, C19.2, C2.2, C20.2, C22.2, C23.2, C24.2, C25.2, C26.2, C27.2, C28.2, C3.2, C30.2, C4.2, C5.2, C6.2, C7.2, C8.2, D1.2 (A2), D3.1 (K), D4.1 (K), D5.1 (K), J1.A1 (GND), J1.A12 (GND), J1.B1 (GND), J1.B12 (GND), J1.SH (SHIELD), J2.A1 (GND), J2.A12 (GND), J2.B1 (GND), J2.B12 (GND), J2.SH (SHIELD), J3.2 (Pin_2), J4.2 (Pin_2), J5.2 (Pin_2), J6.2 (Pin_2), Q1.2 (S), Q2.2 (S), R1.2, R12.2, R14.2, R16.2, R2.2, R24.2, R3.2, R4.2, R7.2, R8.2, SW1.2, TP24.1, TP25.1, TP26.1, TP27.1, U1.11 (GND), U2.10 (ACDRV2), U2.11 (ACDRV1), U2.27 (GND), U3.13 (PGND), U3.8 (AGND), U4.13 (GND), U4.18 (GND), U4.23 (GND), U4.28 (GND), U4.3 (GND), U4.33 (AGND), U4.38 (GND), U4.8 (GND)
- new net HISET: R2.1, U1.9 (ISET)
- new net HVSET: R1.1, U1.8 (VSET)
- new net INT: R10.1, TP11.1, U2.21 (INT), U4.9 (GPIO6)
- new net LEDA0: D3.2 (A), R21.2
- new net LEDA1: D4.2 (A), R22.2
- new net LEDA2: D5.2 (A), R23.2
- new net LED_BAT: R22.1, U4.22 (GPIO17)
- new net LED_FLT: R23.1, U4.24 (GPIO18)
- new net LED_PWR: R21.1, U4.21 (GPIO16)
- new net PACK_P: J3.1 (Pin_1), JP3.1 (A), R5.1, TP12.1
- new net PG: R15.1, TP17.1, U3.5 (PG), U4.11 (GPIO8)
- new net PICO_VSYS: D2.1 (K), U4.39 (VSYS)
- new net PI_PWR_BTN: J5.1 (Pin_1), Q2.3 (D)
- new net PMID: C5.1, C6.1, C7.1, C8.1, TP2.1, U2.29 (PMID)
- new net PROG: R3.1, U2.20 (PROG)
- new net PWR_BTN: Q2.1 (G), R24.1, U4.19 (GPIO14)
- new net QON: TP7.1, U2.12 (QON)
- new net REGN: C11.1, R6.1, TP5.1, U2.17 (ILIM_HIZ), U2.5 (REGN)
- new net RUN: TP23.1, U4.30 (RUN)
- new net SCL: J7.2 (Pin_2), R20.1, TP22.1, U1.7 (SCL), U2.14 (SCL), U4.7 (GPIO5)
- new net SDA: J7.1 (Pin_1), R19.1, TP21.1, U1.6 (SDA), U2.15 (SDA), U4.6 (GPIO4)
- new net SDRV: C20.1, U2.24 (SDRV)
- new net STAT: R9.1, TP10.1, U2.1 (STAT), U4.10 (GPIO7)
- new net SW1: C9.2, L1.1, TP3.1, U2.28 (SW1)
- new net SW2: C10.2, L1.2, TP4.1, U2.26 (SW2)
- new net SW_B: C21.2, L2.1, TP13.1, U3.1 (SW), U3.2 (SW), U3.3 (SW)
- new net TS: J6.1 (Pin_1), R6.2, R7.1, R8.1, TP6.1, U2.16 (TS)
- new net USER_BTN: SW1.1, U4.25 (GPIO19)
- new net V5: C30.1, D2.2 (A), J2.A4 (VBUS), J2.A9 (VBUS), J2.B4 (VBUS), J2.B9 (VBUS), J4.1 (Pin_1), JP2.2 (B), R17.1, R18.1, TP19.1
- new net V5_B: C25.1, C26.1, C27.1, C28.1, C29.1, JP2.1 (A), L2.2, R11.1, TP15.1
- new net VBUS: C1.1, C2.1, C3.1, C4.1, D1.1 (A1), F1.2, TP1.1, U1.1 (VIN), U2.2 (VBUS), U2.3 (VBUS), U2.8 (VAC2), U2.9 (VAC1)
- new net VBUS_RAW: F1.1, J1.A4 (VBUS), J1.A9 (VBUS), J1.B4 (VBUS), J1.B9 (VBUS)
- new net VSYS: C12.1, C13.1, C14.1, C15.1, C16.1, C17.1, JP1.1 (A), TP8.1, U2.25 (SYS)
- new net VSYS_B: C22.1, C23.1, C24.1, JP1.2 (B), R13.1, TP18.1, U3.10 (VIN), U3.11 (VIN), U3.12 (VIN)
- no-connect marks 0 -> 30
Other:
- note added: "1 Input / PD sink"
- note added: "2 Charger BQ25792"
- note added: "3 Pack and links"
- note added: "4 5V buck LMR51450"
- note added: "5 Output"
- note added: "6 MCU (Pico module)"
- note added: "7 Mechanical"
- note added: "Generated by hardware/kicad/gen/gen_sch.py from design.py - edit design.py, not this file. See hardware/DECISIONS.md."
- note removed: "SUB-CIRCUIT 1: USB-PD SINK & INRUSH PROTECTION (HUSB238 + SMAJ24A + DMP3010LK3)"
- note removed: "SUB-CIRCUIT 2: 2S BATTERY BMS & BALANCING (HY2120-LB + DUAL AO8822 + HY2212)"
- note removed: "SUB-CIRCUIT 3: 2S SWITCHING CHARGER & POWER PATH (MP2762A + 2.2uH INDUCTOR)"
- note removed: "SUB-CIRCUIT 4: 5.1V @ 5A SYNCHRONOUS BUCK-BOOST (TPS55289 + 1.5uH + POLYMER CAPS)"
- note removed: "SUB-CIRCUIT 5: RASPBERRY PI 5 USB-C HOST INTERFACE & PWR_BTN HEADER"
- note removed: "SUB-CIRCUIT 6: RP2040 MCU, 16MB FLASH, 3.3V LDO & ANALOG SENSE DIVIDERS"
- company: Web3 Pi Open Hardware -> Pi-cemaker
- title: Pi-cemaker: 2S Li-ion UPS for Raspberry Pi 5 -> Pi-cemaker Lite 2S UPS
